Commit message: [UPD] allow import kachaka urdf model to other files

File: ros2/kachaka_description/robot/kachaka.urdf.xacro (robot description, xacro)
@@ -13,4 +13,5 @@
     <color rgba="0.0 0.0 0.0 1.0" />
   </material>
+  <xacro:macro name="kachaka_robot" params="parent *origin">
   <link name="base_footprint" />
   <link name="base_link">
@@ -232,4 +233,5 @@
     <parent link="base_footprint" />
     <child link="base_link" />
+    <xacro:insert_block name="origin" />
   </joint>
   <joint name="base_r_drive_wheel_joint"
@@ -261,3 +263,4 @@
             xyz="0.0756 -0.0655 0.05146" />
   </joint>
+  </xacro:macro>
 </robot>

Commit message: [UPD] base_footprint from main urdf file

File: ros2/kachaka_description/robot/kachaka.urdf.xacro (robot description, xacro)
@@ -14,5 +14,4 @@
   </material>
   <xacro:macro name="kachaka_robot" params="parent *origin">
-  <link name="base_footprint" />
   <link name="base_link">
     <inertial>
@@ -231,5 +230,5 @@
   <joint name="base_footprint_joint"
          type="fixed">
-    <parent link="base_footprint" />
+    <parent link="${parent}" />
     <child link="base_link" />
     <xacro:insert_block name="origin" />

Commit message: [FIX] indent

File: ros2/kachaka_description/robot/kachaka.urdf.xacro (robot description, xacro)
@@ -14,252 +14,252 @@
   </material>
   <xacro:macro name="kachaka_robot" params="parent *origin">
-  <link name="base_link">
-    <inertial>
-      <mass value="6.4" />
-      <origin xyz="0 0 0"
-              rpy="0 0 0" />
-      <inertia ixx="2.1342e-02"
-               ixy="0"
-               ixz="0"
-               iyy="2.1342e-02"
-               iyz="0"
-               izz="4.2667e-02" />
-    </inertial>
-    <visual>
-      <origin xyz="0.0435 0.0 0.0475"
-              rpy="0 0 0" />
-      <geometry>
-        <box size="0.387 0.240 0.095" />
-      </geometry>
-      <material name="body" />
-    </visual>
-    <collision>
-      <origin xyz="0.0435 0.0 0.0475"
-              rpy="0 0 0" />
-      <geometry>
-        <box size="0.387 0.240 0.095" />
-      </geometry>
-      <material name="body" />
-    </collision>
-  </link>
-  <joint name="lidar_joint"
-         type="fixed">
-    <parent link="base_link" />
-    <child link="laser_frame" />
-    <origin rpy="0 0 ${PI / 2.0}"
-            xyz="0.156 0 0.1049" />
-  </joint>
-  <joint name="docking_joint"
-         type="prismatic">
-    <parent link="base_link" />
-    <child link="docking_link" />
-    <axis xyz="0 0 1.0" />
-    <origin rpy="0 0 0"
-            xyz="0 0 0" />
-    <limit lower="0.0"
-           upper="0.012"
-           effort="1.0"
-           velocity="1.0" />
-  </joint>
-  <joint name="camera_front_joint"
-         type="fixed">
-    <parent link="base_link" />
-    <child link="camera_front_link" />
-    <origin rpy="-${PI / 2.0} 0 -${PI / 2.0}"
-            xyz="${0.2196 - 0.01} 0 0.070" />
-  </joint>
-  <joint name="camera_back_joint"
-         type="fixed">
-    <parent link="base_link" />
-    <child link="camera_back_link" />
-    <origin rpy="-${PI / 2.0} 0 ${PI / 2.0}"
-            xyz="${-0.150 + 0.01} 0 0.070" />
-  </joint>
-  <joint name="tof_joint"
-         type="fixed">
-    <parent link="base_link" />
-    <child link="tof_link" />
-    <origin rpy="-${PI / 4.0} 0 -${PI / 2.0}"
-            xyz="0.221 0.0 0.0418" />
-  </joint>
-  <link name="base_r_drive_wheel_link">
-    <inertial>
-      <mass value="0.2" />
-      <origin xyz="0 0 0"
-              rpy="0 0 0" />
-      <inertia ixx="0.001"
-               ixy="0"
-               ixz="0"
-               iyy="0.001"
-               iyz="0"
-               izz="0.001" />
-    </inertial>
-    <visual>
-      <origin xyz="0 0 0"
-              rpy="${PI / 2.0} 0 0" />
-      <geometry>
-        <cylinder length="0.025"
-                  radius="0.045" />
-      </geometry>
-      <material name="tire" />
-    </visual>
-    <collision>
-      <origin xyz="0 0 0"
-              rpy="${PI / 2.0} 0 0" />
-      <geometry>
-        <cylinder length="0.025"
-                  radius="0.045" />
-      </geometry>
-      <material name="tire" />
-    </collision>
-  </link>
-  <link name="laser_frame">
-    <inertial>
-      <mass value="0.2" />
-      <origin xyz="0 0 0"
-              rpy="0 0 0" />
-      <inertia ixx="0.001"
-               ixy="0"
-               ixz="0"
-               iyy="0.001"
-               iyz="0"
-               izz="0.001" />
-    </inertial>
-  </link>
-  <link name="docking_link">
-    <inertial>
-      <mass value="0.2" />
-      <origin xyz="0 0 0"
-              rpy="0 0 0" />
-      <inertia ixx="0.001"
-               ixy="0"
-               ixz="0"
-               iyy="0.001"
-               iyz="0"
-               izz="0.001" />
-    </inertial>
-    <visual>
-      <origin xyz="0 0 0.1075"
-              rpy="0 0 0" />
-      <geometry>
-        <cylinder length="0.015"
-                  radius="0.025" />
-      </geometry>
-      <material name="body" />
-    </visual>
-    <collision>
-      <origin xyz="0 0 0.1075"
-              rpy="0 0 0" />
-      <geometry>
-        <cylinder length="0.015"
-                  radius="0.025" />
-      </geometry>
-      <material name="body" />
-    </collision>
-  </link>
-  <link name="camera_front_link">
-    <inertial>
-      <mass value="0.2" />
-      <origin xyz="0 0 0"
-              rpy="0 0 0" />
-      <inertia ixx="0.001"
-               ixy="0"
-               ixz="0"
-               iyy="0.001"
-               iyz="0"
-               izz="0.001" />
-    </inertial>
-  </link>
-  <link name="camera_back_link">
-    <inertial>
-      <mass value="0.2" />
-      <origin xyz="0 0 0"
-              rpy="0 0 0" />
-      <inertia ixx="0.001"
-               ixy="0"
-               ixz="0"
-               iyy="0.001"
-               iyz="0"
-               izz="0.001" />
-    </inertial>
-  </link>
-  <link name="tof_link">
-    <inertial>
-      <mass value="0.2" />
-      <origin xyz="0 0 0"
-              rpy="0 0 0" />
-      <inertia ixx="0.001"
-               ixy="0"
-               ixz="0"
-               iyy="0.001"
-               iyz="0"
-               izz="0.001" />
-    </inertial>
-  </link>
-  <link name="base_l_drive_wheel_link">
-    <inertial>
-      <mass value="0.2" />
-      <origin xyz="0 0 0"
-              rpy="0 0 0" />
-      <inertia ixx="0.001"
-               ixy="0"
-               ixz="0"
-               iyy="0.001"
-               iyz="0"
-               izz="0.001" />
-    </inertial>
-    <visual>
-      <origin xyz="0 0 0"
-              rpy="${PI / 2.0} 0 0" />
-      <geometry>
-        <cylinder length="0.025"
-                  radius="0.045" />
-      </geometry>
-      <material name="tire" />
-    </visual>
-    <collision>
-      <origin xyz="0 0 0"
-              rpy="${PI / 2.0} 0 0" />
-      <geometry>
-        <cylinder length="0.025"
-                  radius="0.045" />
-      </geometry>
-      <material name="tire" />
-    </collision>
-  </link>
-  <joint name="base_footprint_joint"
-         type="fixed">
-    <parent link="${parent}" />
-    <child link="base_link" />
-    <xacro:insert_block name="origin" />
-  </joint>
-  <joint name="base_r_drive_wheel_joint"
-         type="continuous">
-    <parent link="base_link" />
-    <child link="base_r_drive_wheel_link" />
-    <origin rpy="0 0 0"
-            xyz="0.0 -0.100 0.045" />
-    <axis xyz="0 1 0" />
-    <limit velocity="10"
-           effort="100" />
-  </joint>
-  <joint name="base_l_drive_wheel_joint"
-         type="continuous">
-    <parent link="base_link" />
-    <child link="base_l_drive_wheel_link" />
-    <origin rpy="0 0 0"
-            xyz="0.0 0.100 0.045" />
-    <axis xyz="0 1 0" />
-    <limit velocity="10"
-           effort="100" />
-  </joint>
-  <link name="imu_link" />
-  <joint name="imu_joint"
-         type="fixed">
-    <parent link="base_link" />
-    <child link="imu_link" />
-    <origin rpy="0 0 0"
-            xyz="0.0756 -0.0655 0.05146" />
-  </joint>
+    <link name="base_link">
+      <inertial>
+        <mass value="6.4" />
+        <origin xyz="0 0 0"
+                rpy="0 0 0" />
+        <inertia ixx="2.1342e-02"
+                ixy="0"
+                ixz="0"
+                iyy="2.1342e-02"
+                iyz="0"
+                izz="4.2667e-02" />
+      </inertial>
+      <visual>
+        <origin xyz="0.0435 0.0 0.0475"
+                rpy="0 0 0" />
+        <geometry>
+          <box size="0.387 0.240 0.095" />
+        </geometry>
+        <material name="body" />
+      </visual>
+      <collision>
+        <origin xyz="0.0435 0.0 0.0475"
+                rpy="0 0 0" />
+        <geometry>
+          <box size="0.387 0.240 0.095" />
+        </geometry>
+        <material name="body" />
+      </collision>
+    </link>
+    <joint name="lidar_joint"
+          type="fixed">
+      <parent link="base_link" />
+      <child link="laser_frame" />
+      <origin rpy="0 0 ${PI / 2.0}"
+              xyz="0.156 0 0.1049" />
+    </joint>
+    <joint name="docking_joint"
+          type="prismatic">
+      <parent link="base_link" />
+      <child link="docking_link" />
+      <axis xyz="0 0 1.0" />
+      <origin rpy="0 0 0"
+              xyz="0 0 0" />
+      <limit lower="0.0"
+            upper="0.012"
+            effort="1.0"
+            velocity="1.0" />
+    </joint>
+    <joint name="camera_front_joint"
+          type="fixed">
+      <parent link="base_link" />
+      <child link="camera_front_link" />
+      <origin rpy="-${PI / 2.0} 0 -${PI / 2.0}"
+              xyz="${0.2196 - 0.01} 0 0.070" />
+    </joint>
+    <joint name="camera_back_joint"
+          type="fixed">
+      <parent link="base_link" />
+      <child link="camera_back_link" />
+      <origin rpy="-${PI / 2.0} 0 ${PI / 2.0}"
+              xyz="${-0.150 + 0.01} 0 0.070" />
+    </joint>
+    <joint name="tof_joint"
+          type="fixed">
+      <parent link="base_link" />
+      <child link="tof_link" />
+      <origin rpy="-${PI / 4.0} 0 -${PI / 2.0}"
+              xyz="0.221 0.0 0.0418" />
+    </joint>
+    <link name="base_r_drive_wheel_link">
+      <inertial>
+        <mass value="0.2" />
+        <origin xyz="0 0 0"
+                rpy="0 0 0" />
+        <inertia ixx="0.001"
+                ixy="0"
+                ixz="0"
+                iyy="0.001"
+                iyz="0"
+                izz="0.001" />
+      </inertial>
+      <visual>
+        <origin xyz="0 0 0"
+                rpy="${PI / 2.0} 0 0" />
+        <geometry>
+          <cylinder length="0.025"
+                    radius="0.045" />
+        </geometry>
+        <material name="tire" />
+      </visual>
+      <collision>
+        <origin xyz="0 0 0"
+                rpy="${PI / 2.0} 0 0" />
+        <geometry>
+          <cylinder length="0.025"
+                    radius="0.045" />
+        </geometry>
+        <material name="tire" />
+      </collision>
+    </link>
+    <link name="laser_frame">
+      <inertial>
+        <mass value="0.2" />
+        <origin xyz="0 0 0"
+                rpy="0 0 0" />
+        <inertia ixx="0.001"
+                ixy="0"
+                ixz="0"
+                iyy="0.001"
+                iyz="0"
+                izz="0.001" />
+      </inertial>
+    </link>
+    <link name="docking_link">
+      <inertial>
+        <mass value="0.2" />
+        <origin xyz="0 0 0"
+                rpy="0 0 0" />
+        <inertia ixx="0.001"
+                ixy="0"
+                ixz="0"
+                iyy="0.001"
+                iyz="0"
+                izz="0.001" />
+      </inertial>
+      <visual>
+        <origin xyz="0 0 0.1075"
+                rpy="0 0 0" />
+        <geometry>
+          <cylinder length="0.015"
+                    radius="0.025" />
+        </geometry>
+        <material name="body" />
+      </visual>
+      <collision>
+        <origin xyz="0 0 0.1075"
+                rpy="0 0 0" />
+        <geometry>
+          <cylinder length="0.015"
+                    radius="0.025" />
+        </geometry>
+        <material name="body" />
+      </collision>
+    </link>
+    <link name="camera_front_link">
+      <inertial>
+        <mass value="0.2" />
+        <origin xyz="0 0 0"
+                rpy="0 0 0" />
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
Commit message: [UPD] move property inside macro

File: ros2/kachaka_description/robot/kachaka.urdf.xacro (robot description, xacro)
@@ -2,6 +2,4 @@
 <robot name="kachaka"
        xmlns:xacro="http://ros.org/wiki/xacro">
-  <xacro:property name="PI"
-                  value="3.141592653589793" />
   <material name="body">
     <color rgba="0.2175 0.2355 0.246 1.0" />
@@ -14,4 +12,6 @@
   </material>
   <xacro:macro name="kachaka_robot" params="parent *origin">
+    <xacro:property name="PI"
+                    value="3.141592653589793" />
     <link name="base_link">
       <inertial>

Commit message: [UPD] delete materials from main xacro file

File: ros2/kachaka_description/robot/kachaka.urdf.xacro (robot description, xacro)
@@ -2,13 +2,4 @@
 <robot name="kachaka"
        xmlns:xacro="http://ros.org/wiki/xacro">
-  <material name="body">
-    <color rgba="0.2175 0.2355 0.246 1.0" />
-  </material>
-  <material name="tire">
-    <color rgba="0.3 0.3 0.3 1.0" />
-  </material>
-  <material name="black">
-    <color rgba="0.0 0.0 0.0 1.0" />
-  </material>
   <xacro:macro name="kachaka_robot" params="parent *origin">
     <xacro:property name="PI"

Commit message: [FIX] inertia based on primitive shapes

File: ros2/kachaka_description/robot/kachaka.urdf.xacro (robot description, xacro)
@@ -85,57 +85,41 @@
   <link name="base_r_drive_wheel_link">
     <inertial>
-      <mass value="0.2" />
-      <origin xyz="0 0 0"
-              rpy="0 0 0" />
-      <inertia ixx="0.001"
-               ixy="0"
-               ixz="0"
-               iyy="0.001"
-               iyz="0"
-               izz="0.001" />
-    </inertial>
-    <visual>
-      <origin xyz="0 0 0"
-              rpy="${PI / 2.0} 0 0" />
-      <geometry>
-        <cylinder length="0.025"
-                  radius="0.045" />
-      </geometry>
-      <material name="tire" />
-    </visual>
-    <collision>
-      <origin xyz="0 0 0"
-              rpy="${PI / 2.0} 0 0" />
-      <geometry>
-        <cylinder length="0.025"
-                  radius="0.045" />
-      </geometry>
-      <material name="tire" />
-    </collision>
-  </link>
-  <link name="laser_frame">
-    <inertial>
-      <mass value="0.2" />
-      <origin xyz="0 0 0"
-              rpy="0 0 0" />
-      <inertia ixx="0.001"
-               ixy="0"
-               ixz="0"
-               iyy="0.001"
-               iyz="0"
-               izz="0.001" />
-    </inertial>
-  </link>
+      <mass value="0.2" /> <!-- TODO - Update mass value -->
+      <origin xyz="0 0 0"
+              rpy="${PI / 2.0} 0 0" />
+      <!-- Bug - inertial rotation is not reflected in Rviz2 -->
+      <!-- https://github.com/ros2/rviz/pull/1171 -->
+      <inertia ixx="${1/12*0.2*(3*0.045**2+0.025**2)}" ixy="0" ixz="0"
+               iyy="${1/12*0.2*(3*0.045**2+0.025**2)}" iyz="0"
+               izz="${1/2*0.2*(0.045**2)}" />
+    </inertial>
+    <visual>
+      <origin xyz="0 0 0"
+              rpy="${PI / 2.0} 0 0" />
+      <geometry>
+        <cylinder length="0.025"
+                  radius="0.045" />
+      </geometry>
+      <material name="tire" />
+    </visual>
+    <collision>
+      <origin xyz="0 0 0"
+              rpy="${PI / 2.0} 0 0" />
+      <geometry>
+        <cylinder length="0.025"
+                  radius="0.045" />
+      </geometry>
+      <material name="tire" />
+    </collision>
+  </link>
+  <link name="laser_frame" />
   <link name="docking_link">
     <inertial>
-      <mass value="0.2" />
-      <origin xyz="0 0 0"
-              rpy="0 0 0" />
-      <inertia ixx="0.001"
-               ixy="0"
-               ixz="0"
-               iyy="0.001"
-               iyz="0"
-               izz="0.001" />
+      <mass value="0.2" /> <!-- TODO - Update mass value -->
+      <origin xyz="0 0 0.1075"
+              rpy="0 0 0" />
+      <inertia ixx="${1/12*0.2*(3*0.025**2+0.015**2)}" ixy="0" ixz="0"
+               iyy="${1/12*0.2*(3*0.025**2+0.015**2)}" iyz="0"
+               izz="${1/2*0.2*(0.025**2)}" />
     </inertial>
     <visual>
@@ -201,11 +185,10 @@
       <mass value="0.2" />
       <origin xyz="0 0 0"
-              rpy="0 0 0" />
-      <inertia ixx="0.001"
-               ixy="0"
-               ixz="0"
-               iyy="0.001"
-               iyz="0"
-               izz="0.001" />
+              rpy="${PI / 2.0} 0 0" />
+      <!-- Bug - inertial rotation is not reflected in Rviz2 -->
+      <!-- https://github.com/ros2/rviz/pull/1171 -->
+      <inertia ixx="${1/12*0.2*(3*0.045**2+0.025**2)}" ixy="0" ixz="0"
+               iyy="${1/12*0.2*(3*0.045**2+0.025**2)}" iyz="0"
+               izz="${1/2*0.2*(0.045**2)}" />
     </inertial>
     <visual>

Commit message: [DEL] remove not implemented inertias

File: ros2/kachaka_description/robot/kachaka.urdf.xacro (robot description, xacro)
@@ -142,43 +142,7 @@
     </collision>
   </link>
-  <link name="camera_front_link">
-    <inertial>
-      <mass value="0.2" />
-      <origin xyz="0 0 0"
-              rpy="0 0 0" />
-      <inertia ixx="0.001"
-               ixy="0"
-               ixz="0"
-               iyy="0.001"
-               iyz="0"
-               izz="0.001" />
-    </inertial>
-  </link>
-  <link name="camera_back_link">
-    <inertial>
-      <mass value="0.2" />
-      <origin xyz="0 0 0"
-              rpy="0 0 0" />
-      <inertia ixx="0.001"
-               ixy="0"
-               ixz="0"
-               iyy="0.001"
-               iyz="0"
-               izz="0.001" />
-    </inertial>
-  </link>
-  <link name="tof_link">
-    <inertial>
-      <mass value="0.2" />
-      <origin xyz="0 0 0"
-              rpy="0 0 0" />
-      <inertia ixx="0.001"
-               ixy="0"
-               ixz="0"
-               iyy="0.001"
-               iyz="0"
-               izz="0.001" />
-    </inertial>
-  </link>
+  <link name="camera_front_link" />
+  <link name="camera_back_link" />
+  <link name="tof_link" />
   <link name="base_l_drive_wheel_link">
     <inertial>

Commit message: [FIX] robot mass and inertia

File: ros2/kachaka_description/robot/kachaka.urdf.xacro (robot description, xacro)
@@ -16,13 +16,10 @@
   <link name="base_link">
     <inertial>
-      <mass value="6.4" />
-      <origin xyz="0 0 0"
-              rpy="0 0 0" />
-      <inertia ixx="2.1342e-02"
-               ixy="0"
-               ixz="0"
-               iyy="2.1342e-02"
-               iyz="0"
-               izz="4.2667e-02" />
+      <mass value="10" />
+      <origin xyz="0 0 0"
+              rpy="0 0 0" />
+      <inertia ixx="${1/12*10*(0.095**2+0.240**2)}" ixy="0" ixz="0"
+               iyy="${1/12*10*(0.095**2+0.387**2)}" iyz="0"
+               izz="${1/12*10*(0.387**2+0.240**2)}" />
     </inertial>
     <visual>
