Commit message: [ADD] kachaka import method

File: ros2/kachaka_description/robot/kachaka.urdf.xacro (robot description, xacro)
@@ -2,262 +2,10 @@
 <robot name="kachaka"
        xmlns:xacro="http://ros.org/wiki/xacro">
-  <xacro:property name="PI"
-                  value="3.141592653589793" />
-  <material name="body">
-    <color rgba="0.2175 0.2355 0.246 1.0" />
-  </material>
-  <material name="tire">
-    <color rgba="0.3 0.3 0.3 1.0" />
-  </material>
-  <material name="black">
-    <color rgba="0.0 0.0 0.0 1.0" />
-  </material>
+  <xacro:include filename="$(find kachaka_description)/urdf/_materials.urdf.xacro" />
+  <xacro:include filename="$(find kachaka_description)/urdf/_values.urdf.xacro" />
+  <xacro:include filename="$(find kachaka_description)/urdf/_kachaka.urdf.xacro" />
   <link name="base_footprint" />
-  <link name="base_link">
-    <inertial>
-      <mass value="6.4" />
-      <origin xyz="0 0 0"
-              rpy="0 0 0" />
-      <inertia ixx="2.1342e-02"
-               ixy="0"
-               ixz="0"
-               iyy="2.1342e-02"
-               iyz="0"
-               izz="4.2667e-02" />
-    </inertial>
-    <visual>
-      <origin xyz="-0.150 -0.120 0.0"
-              rpy="0 0 0" />
-      <geometry>
-        <mesh filename="package://kachaka_description/meshes/kachaka/body.stl" />
-      </geometry>
-      <material name="body" />
-    </visual>
-    <collision>
-      <origin xyz="0.0435 0.0 0.0475"
-              rpy="0 0 0" />
-      <geometry>
-        <box size="0.387 0.240 0.095" />
-      </geometry>
-      <material name="body" />
-    </collision>
-  </link>
-  <joint name="lidar_joint"
-         type="fixed">
-    <parent link="base_link" />
-    <child link="laser_frame" />
-    <origin rpy="0 0 ${PI / 2.0}"
-            xyz="0.156 0 0.1049" />
-  </joint>
-  <joint name="docking_joint"
-         type="prismatic">
-    <parent link="base_link" />
-    <child link="docking_link" />
-    <axis xyz="0 0 1.0" />
-    <origin rpy="0 0 0"
-            xyz="0 0 0" />
-    <limit lower="0.0"
-           upper="0.012"
-           effort="1.0"
-           velocity="1.0" />
-  </joint>
-  <joint name="camera_front_joint"
-         type="fixed">
-    <parent link="base_link" />
-    <child link="camera_front_link" />
-    <origin rpy="-${PI / 2.0} 0 -${PI / 2.0}"
-            xyz="${0.2196 - 0.01} 0 0.070" />
-  </joint>
-  <joint name="camera_back_joint"
-         type="fixed">
-    <parent link="base_link" />
-    <child link="camera_back_link" />
-    <origin rpy="-${PI / 2.0} 0 ${PI / 2.0}"
-            xyz="${-0.150 + 0.01} 0 0.070" />
-  </joint>
-  <joint name="tof_joint"
-         type="fixed">
-    <parent link="base_link" />
-    <child link="tof_link" />
-    <origin rpy="-${PI / 4.0} 0 -${PI / 2.0}"
-            xyz="0.221 0.0 0.0418" />
-  </joint>
-  <link name="base_r_drive_wheel_link">
-    <inertial>
-      <mass value="0.2" />
-      <origin xyz="0 0 0"
-              rpy="0 0 0" />
-      <inertia ixx="0.001"
-               ixy="0"
-               ixz="0"
-               iyy="0.001"
-               iyz="0"
-               izz="0.001" />
-    </inertial>
-    <visual>
-      <origin xyz="0 0 0"
-              rpy="0 0 0" />
-      <geometry>
-        <mesh filename="package://kachaka_description/meshes/kachaka/right_tire.stl"
-              scale="1.0 1.0 1.0" />
-      </geometry>
-      <material name="tire" />
-    </visual>
-    <collision>
-      <origin xyz="0 0 0"
-              rpy="${PI / 2.0} 0 0" />
-      <geometry>
-        <cylinder length="0.025"
-                  radius="0.045" />
-      </geometry>
-      <material name="tire" />
-    </collision>
-  </link>
-  <link name="laser_frame">
-    <inertial>
-      <mass value="0.2" />
-      <origin xyz="0 0 0"
-              rpy="0 0 0" />
-      <inertia ixx="0.001"
-               ixy="0"
-               ixz="0"
-               iyy="0.001"
-               iyz="0"
-               izz="0.001" />
-    </inertial>
-  </link>
-  <link name="docking_link">
-    <inertial>
-      <mass value="0.2" />
-      <origin xyz="0 0 0"
-              rpy="0 0 0" />
-      <inertia ixx="0.001"
-               ixy="0"
-               ixz="0"
-               iyy="0.001"
-               iyz="0"
-               izz="0.001" />
-    </inertial>
-    <visual>
-      <origin xyz="0 0 0.073"
-              rpy="0 0 0" />
-      <geometry>
-        <mesh filename="package://kachaka_description/meshes/kachaka/solenoid.stl"
-              scale="1.0 1.0 1.0" />
-      </geometry>
-      <material name="body" />
-    </visual>
-    <collision>
-      <origin xyz="0 0 0.1075"
-              rpy="0 0 0" />
-      <geometry>
-        <cylinder length="0.015"
-                  radius="0.025" />
-      </geometry>
-      <material name="body" />
-    </collision>
-  </link>
-  <link name="camera_front_link">
-    <inertial>
-      <mass value="0.2" />
-      <origin xyz="0 0 0"
-              rpy="0 0 0" />
-      <inertia ixx="0.001"
-               ixy="0"
-               ixz="0"
-               iyy="0.001"
-               iyz="0"
-               izz="0.001" />
-    </inertial>
-  </link>
-  <link name="camera_back_link">
-    <inertial>
-      <mass value="0.2" />
-      <origin xyz="0 0 0"
-              rpy="0 0 0" />
-      <inertia ixx="0.001"
-               ixy="0"
-               ixz="0"
-               iyy="0.001"
-               iyz="0"
-               izz="0.001" />
-    </inertial>
-  </link>
-  <link name="tof_link">
-    <inertial>
-      <mass value="0.2" />
-      <origin xyz="0 0 0"
-              rpy="0 0 0" />
-      <inertia ixx="0.001"
-               ixy="0"
-               ixz="0"
-               iyy="0.001"
-               iyz="0"
-               izz="0.001" />
-    </inertial>
-  </link>
-  <link name="base_l_drive_wheel_link">
-    <inertial>
-      <mass value="0.2" />
-      <origin xyz="0 0 0"
-              rpy="0 0 0" />
-      <inertia ixx="0.001"
-               ixy="0"
-               ixz="0"
-               iyy="0.001"
-               iyz="0"
-               izz="0.001" />
-    </inertial>
-    <visual>
-      <origin xyz="0 0 0"
-              rpy="0 0 0" />
-      <geometry>
-        <mesh filename="package://kachaka_description/meshes/kachaka/left_tire.stl"
-              scale="1.0 1.0 1.0" />
-      </geometry>
-      <material name="tire" />
-    </visual>
-    <collision>
-      <origin xyz="0 0 0"
-              rpy="${PI / 2.0} 0 0" />
-      <geometry>
-        <cylinder length="0.025"
-                  radius="0.045" />
-      </geometry>
-      <material name="tire" />
-    </collision>
-  </link>
-  <joint name="base_footprint_joint"
-         type="fixed">
-    <parent link="base_footprint" />
-    <child link="base_link" />
-  </joint>
-  <joint name="base_r_drive_wheel_joint"
-         type="continuous">
-    <parent link="base_link" />
-    <child link="base_r_drive_wheel_link" />
-    <origin rpy="0 0 0"
-            xyz="0.0 -0.100 0.045" />
-    <axis xyz="0 1 0" />
-    <limit velocity="10"
-           effort="100" />
-  </joint>
-  <joint name="base_l_drive_wheel_joint"
-         type="continuous">
-    <parent link="base_link" />
-    <child link="base_l_drive_wheel_link" />
-    <origin rpy="0 0 0"
-            xyz="0.0 0.100 0.045" />
-    <axis xyz="0 1 0" />
-    <limit velocity="10"
-           effort="100" />
-  </joint>
-  <link name="imu_link" />
-  <joint name="imu_joint"
-         type="fixed">
-    <parent link="base_link" />
-    <child link="imu_link" />
-    <origin rpy="0 0 0"
-            xyz="0.0756 -0.0655 0.05146" />
-  </joint>
+  <xacro:kachaka_robot parent="base_footprint">
+    <origin xyz="0 0 0" rpy="0 0 0"/>
+  </xacro:kachaka_robot>
 </robot>
