Commit message: [UPD] xacro-generated urdf

File: ros2/kachaka_description/robot/kachaka.urdf (robot description, URDF)
Before this commit: robot kachaka, 10 links, 9 joints
Joints:
- joint base_footprint_joint: origin (none) -> xyz=0 0 0 rpy=0 0 0

Commit message: [UPD] update urdf file based on xacro

File: ros2/kachaka_description/robot/kachaka.urdf (robot description, URDF)
Before this commit: robot kachaka, 10 links, 9 joints
Links:
- link base_link: mass 6.4 -> 10
- link camera_back_link: mass 0.2 -> None
- link camera_front_link: mass 0.2 -> None
- link laser_frame: mass 0.2 -> None
- link tof_link: mass 0.2 -> None

Commit message: add precise mesh

File: ros2/kachaka_description/robot/kachaka.urdf (robot description, URDF)
Before this commit: robot kachaka, 10 links, 9 joints
Links:
- link base_l_drive_wheel_link: geometry collision cylinder length=0.025 radius=0.045; visual mesh filename=package://kachaka_description/meshes/kachaka/left_tire.stl scale=1.0 1.0 1.0
- link base_link: geometry collision box size=0.387 0.240 0.095; visual mesh filename=package://kachaka_description/meshes/kachaka/body.stl
- link base_r_drive_wheel_link: geometry collision cylinder length=0.025 radius=0.045; visual mesh filename=package://kachaka_description/meshes/kachaka/right_tire.stl scale=1.0 1.0 1.0
- link docking_link: geometry collision cylinder length=0.015 radius=0.025; visual mesh filename=package://kachaka_description/meshes/kachaka/solenoid.stl scale=1.0 1.0 1.0

File: ros2/kachaka_description/robot/kachaka.urdf.xacro (robot description, xacro)
@@ -27,8 +27,8 @@
     </inertial>
     <visual>
-      <origin xyz="0.0435 0.0 0.0475"
-              rpy="0 0 0" />
-      <geometry>
-        <box size="0.387 0.240 0.095" />
+      <origin xyz="-0.150 -0.120 0.0"
+              rpy="0 0 0" />
+      <geometry>
+        <mesh filename="package://kachaka_description/meshes/kachaka/body.stl" />
       </geometry>
       <material name="body" />
@@ -97,4 +97,13 @@
     <visual>
       <origin xyz="0 0 0"
+              rpy="0 0 0" />
+      <geometry>
+        <mesh filename="package://kachaka_description/meshes/kachaka/right_tire.stl"
+              scale="1.0 1.0 1.0" />
+      </geometry>
+      <material name="tire" />
+    </visual>
+    <collision>
+      <origin xyz="0 0 0"
               rpy="${PI / 2.0} 0 0" />
       <geometry>
@@ -103,13 +112,4 @@
       </geometry>
       <material name="tire" />
-    </visual>
-    <collision>
-      <origin xyz="0 0 0"
-              rpy="${PI / 2.0} 0 0" />
-      <geometry>
-        <cylinder length="0.025"
-                  radius="0.045" />
-      </geometry>
-      <material name="tire" />
     </collision>
   </link>
@@ -140,4 +140,13 @@
     </inertial>
     <visual>
+      <origin xyz="0 0 0.073"
+              rpy="0 0 0" />
+      <geometry>
+        <mesh filename="package://kachaka_description/meshes/kachaka/solenoid.stl"
+              scale="1.0 1.0 1.0" />
+      </geometry>
+      <material name="body" />
+    </visual>
+    <collision>
       <origin xyz="0 0 0.1075"
               rpy="0 0 0" />
@@ -147,13 +156,4 @@
       </geometry>
       <material name="body" />
-    </visual>
-    <collision>
-      <origin xyz="0 0 0.1075"
-              rpy="0 0 0" />
-      <geometry>
-        <cylinder length="0.015"
-                  radius="0.025" />
-      </geometry>
-      <material name="body" />
     </collision>
   </link>
@@ -211,8 +211,8 @@
     <visual>
       <origin xyz="0 0 0"
-              rpy="${PI / 2.0} 0 0" />
-      <geometry>
-        <cylinder length="0.025"
-                  radius="0.045" />
+              rpy="0 0 0" />
+      <geometry>
+        <mesh filename="package://kachaka_description/meshes/kachaka/left_tire.stl"
+              scale="1.0 1.0 1.0" />
       </geometry>
       <material name="tire" />

Commit message: [UPD] urdf file with inertia

File: ros2/kachaka_description/robot/kachaka.urdf (robot description, URDF)
Before this commit: robot kachaka, 10 links, 9 joints
Links:
- link base_l_drive_wheel_link: geometry collision cylinder length=0.025 radius=0.045; visual cylinder length=0.025 radius=0.045
- link base_link: mass 6.4 -> 10.0; geometry collision box size=0.387 0.240 0.095; visual box size=0.387 0.240 0.095
- link base_r_drive_wheel_link: geometry collision cylinder length=0.025 radius=0.045; visual cylinder length=0.025 radius=0.045
- link camera_back_link: mass 0.2 -> None
- link camera_front_link: mass 0.2 -> None
- link docking_link: geometry collision cylinder length=0.015 radius=0.025; visual cylinder length=0.015 radius=0.025
- link laser_frame: mass 0.2 -> None
- link tof_link: mass 0.2 -> None
Joints:
- joint base_footprint_joint: origin (none) -> xyz=0 0 0 rpy=0 0 0

Commit message: [FIX] recover stl model

File: ros2/kachaka_description/robot/kachaka.urdf (robot description, URDF)
Before this commit: robot kachaka, 10 links, 9 joints
Links:
- link base_l_drive_wheel_link: geometry collision cylinder length=0.025 radius=0.045; visual mesh filename=file:///home/sobits/colcon_ws/install/kachaka_description/s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 scale=1.0 1.0 1.0
- link base_link: geometry collision box size=0.387 0.240 0.095; visual mesh filename=file:///home/sobits/colcon_ws/install/kachaka_description/s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
- link base_r_drive_wheel_link: geometry collision cylinder length=0.025 radius=0.045; visual mesh filename=file:///home/sobits/colcon_ws/install/kachaka_description/s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 scale=1.0 1.0 1.0
- link docking_link: geometry collision cylinder length=0.015 radius=0.025; visual mesh filename=file:///home/sobits/colcon_ws/install/kachaka_description/s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 scale=1.0 1.0 1.0
