Commit message: [ADD] inertia values

File: ros2/kachaka_description/urdf/_kachaka.urdf.xacro (robot description, xacro)
@@ -5,13 +5,10 @@
     <link name="base_link">
       <inertial>
-        <mass value="6.4" />
-        <origin xyz="0 0 0"
-                rpy="0 0 0" />
-        <inertia ixx="2.1342e-02"
-                ixy="0"
-                ixz="0"
-                iyy="2.1342e-02"
-                iyz="0"
-                izz="4.2667e-02" />
+        <mass value="10.0" />
+        <origin xyz="0 0 0"
+                rpy="0 0 0" />
+        <inertia ixx="${1/12*10*(0.095**2+0.240**2)}" ixy="0" ixz="0"
+                iyy="${1/12*10*(0.095**2+0.387**2)}" iyz="0"
+                izz="${1/12*10*(0.387**2+0.240**2)}" />
       </inertial>
       <visual>
@@ -74,13 +71,12 @@
     <link name="base_r_drive_wheel_link">
       <inertial>
-        <mass value="0.2" />
-        <origin xyz="0 0 0"
-                rpy="0 0 0" />
-        <inertia ixx="0.001"
-                ixy="0"
-                ixz="0"
-                iyy="0.001"
-                iyz="0"
-                izz="0.001" />
+        <mass value="0.2" /> <!-- TODO - Update mass value -->
+        <origin xyz="0 0 0"
+                rpy="${PI / 2.0} 0 0" />
+        <!-- Bug - inertial rotation is not reflected in Rviz2 -->
+        <!-- https://github.com/ros2/rviz/pull/1316 -->
+        <inertia ixx="${1/12*0.2*(3*0.045**2+0.025**2)}" ixy="0" ixz="0"
+                iyy="${1/12*0.2*(3*0.045**2+0.025**2)}" iyz="0"
+                izz="${1/2*0.2*(0.045**2)}" />
       </inertial>
       <visual>
@@ -118,13 +114,10 @@
     <link name="docking_link">
       <inertial>
-        <mass value="0.2" />
-        <origin xyz="0 0 0"
-                rpy="0 0 0" />
-        <inertia ixx="0.001"
-                ixy="0"
-                ixz="0"
-                iyy="0.001"
-                iyz="0"
-                izz="0.001" />
+        <mass value="0.2" /> <!-- TODO - Update mass value -->
+        <origin xyz="0 0 0.1075"
+                rpy="0 0 0" />
+        <inertia ixx="${1/12*0.2*(3*0.025**2+0.015**2)}" ixy="0" ixz="0"
+                iyy="${1/12*0.2*(3*0.025**2+0.015**2)}" iyz="0"
+                izz="${1/2*0.2*(0.025**2)}" />
       </inertial>
       <visual>
@@ -190,11 +183,10 @@
         <mass value="0.2" />
         <origin xyz="0 0 0"
-                rpy="0 0 0" />
-        <inertia ixx="0.001"
-                ixy="0"
-                ixz="0"
-                iyy="0.001"
-                iyz="0"
-                izz="0.001" />
+                rpy="${PI / 2.0} 0 0" />
+        <!-- Bug - inertial rotation is not reflected in Rviz2 -->
+        <!-- https://github.com/ros2/rviz/pull/1171 -->
+        <inertia ixx="${1/12*0.2*(3*0.045**2+0.025**2)}" ixy="0" ixz="0"
+                iyy="${1/12*0.2*(3*0.045**2+0.025**2)}" iyz="0"
+                izz="${1/2*0.2*(0.045**2)}" />
       </inertial>
       <visual>

Commit message: [DEL] not applied inertias

File: ros2/kachaka_description/urdf/_kachaka.urdf.xacro (robot description, xacro)
@@ -99,16 +99,5 @@
       </collision>
     </link>
-    <link name="laser_frame">
-      <inertial>
-        <mass value="0.2" />
-        <origin xyz="0 0 0"
-                rpy="0 0 0" />
-        <inertia ixx="0.001"
-                ixy="0"
-                ixz="0"
-                iyy="0.001"
-                iyz="0"
-                izz="0.001" />
-      </inertial>
+    <link name="laser_frame" />
     </link>
     <link name="docking_link">
@@ -140,43 +129,7 @@
       </collision>
     </link>
-    <link name="camera_front_link">
-      <inertial>
-        <mass value="0.2" />
-        <origin xyz="0 0 0"
-                rpy="0 0 0" />
-        <inertia ixx="0.001"
-                ixy="0"
-                ixz="0"
-                iyy="0.001"
-                iyz="0"
-                izz="0.001" />
-      </inertial>
-    </link>
-    <link name="camera_back_link">
-      <inertial>
-        <mass value="0.2" />
-        <origin xyz="0 0 0"
-                rpy="0 0 0" />
-        <inertia ixx="0.001"
-                ixy="0"
-                ixz="0"
-                iyy="0.001"
-                iyz="0"
-                izz="0.001" />
-      </inertial>
-    </link>
-    <link name="tof_link">
-      <inertial>
-        <mass value="0.2" />
-        <origin xyz="0 0 0"
-                rpy="0 0 0" />
-        <inertia ixx="0.001"
-                ixy="0"
-                ixz="0"
-                iyy="0.001"
-                iyz="0"
-                izz="0.001" />
-      </inertial>
-    </link>
+    <link name="camera_front_link" />
+    <link name="camera_back_link" />
+    <link name="tof_link" />
     <link name="base_l_drive_wheel_link">
       <inertial>

Commit message: [FIX] inertia pose

File: ros2/kachaka_description/urdf/_kachaka.urdf.xacro (robot description, xacro)
@@ -6,5 +6,5 @@
       <inertial>
         <mass value="10.0" />
-        <origin xyz="0 0 0"
+        <origin xyz="0.0435 0.0 0.0475"
                 rpy="0 0 0" />
         <inertia ixx="${1/12*10*(0.095**2+0.240**2)}" ixy="0" ixz="0"
@@ -100,5 +100,4 @@
     </link>
     <link name="laser_frame" />
-    </link>
     <link name="docking_link">
       <inertial>
@@ -107,6 +106,6 @@
                 rpy="0 0 0" />
         <inertia ixx="${1/12*0.2*(3*0.025**2+0.015**2)}" ixy="0" ixz="0"
-                iyy="${1/12*0.2*(3*0.025**2+0.015**2)}" iyz="0"
-                izz="${1/2*0.2*(0.025**2)}" />
+                 iyy="${1/12*0.2*(3*0.025**2+0.015**2)}" iyz="0"
+                 izz="${1/2*0.2*(0.025**2)}" />
       </inertial>
       <visual>

Commit message: [FIX] recover stl model

File: ros2/kachaka_description/urdf/_kachaka.urdf.xacro (robot description, xacro)
@@ -13,8 +13,8 @@
       </inertial>
       <visual>
-        <origin xyz="0.0435 0.0 0.0475"
+        <origin xyz="-0.150 -0.120 0.0"
                 rpy="0 0 0" />
         <geometry>
-          <box size="0.387 0.240 0.095" />
+          <mesh filename="file://$(find kachaka_description)/meshes/kachaka/body.stl"/>
         </geometry>
         <material name="body" />
@@ -82,8 +82,7 @@
       <visual>
         <origin xyz="0 0 0"
-                rpy="${PI / 2.0} 0 0" />
+                rpy="0 0 0" />
         <geometry>
-          <cylinder length="0.025"
-                    radius="0.045" />
+          <mesh filename="file://$(find kachaka_description)/meshes/kachaka/right_tire.stl" scale="1.0 1.0 1.0"/>
         </geometry>
         <material name="tire" />
@@ -110,9 +109,8 @@
       </inertial>
       <visual>
-        <origin xyz="0 0 0.1075"
+        <origin xyz="0 0 0.073"
                 rpy="0 0 0" />
         <geometry>
-          <cylinder length="0.015"
-                    radius="0.025" />
+          <mesh filename="file://$(find kachaka_description)/meshes/kachaka/solenoid.stl" scale="1.0 1.0 1.0"/>
         </geometry>
         <material name="body" />
@@ -144,8 +142,7 @@
       <visual>
         <origin xyz="0 0 0"
-                rpy="${PI / 2.0} 0 0" />
+                rpy="0 0 0" />
         <geometry>
-          <cylinder length="0.025"
-                    radius="0.045" />
+          <mesh filename="file://$(find kachaka_description)/meshes/kachaka/left_tire.stl" scale="1.0 1.0 1.0"/>
         </geometry>
         <material name="tire" />

Commit message: fix robot meshes

File: ros2/kachaka_description/urdf/_kachaka.urdf.xacro (robot description, xacro)
@@ -13,9 +13,8 @@
       </inertial>
       <visual>
-        <origin xyz="0.0435 0.0 0.0475"
-                rpy="0 0 0" />
-        <geometry>
-          <box size="0.387 0.240 0.095" />
-        </geometry>
+	<origin rpy="0 0 0" xyz="-0.150 -0.120 0.0"/>
+	<geometry>
+          <mesh filename="package://kachaka_description/meshes/kachaka/body.stl"/>
+	</geometry>
         <material name="body" />
       </visual>
@@ -81,9 +80,7 @@
       </inertial>
       <visual>
-        <origin xyz="0 0 0"
-                rpy="${PI / 2.0} 0 0" />
+	<origin rpy="0 0 0" xyz="0 0 0"/>
         <geometry>
-          <cylinder length="0.025"
-                    radius="0.045" />
+          <mesh filename="package://kachaka_description/meshes/kachaka/right_tire.stl" scale="1.0 1.0 1.0"/>
         </geometry>
         <material name="tire" />
@@ -110,10 +107,8 @@
       </inertial>
       <visual>
-        <origin xyz="0 0 0.1075"
-                rpy="0 0 0" />
-        <geometry>
-          <cylinder length="0.015"
-                    radius="0.025" />
-        </geometry>
+	<geometry>
+          <mesh filename="package://kachaka_description/meshes/kachaka/solenoid.stl"
+		scale="1.0 1.0 1.0" />
+	</geometry>
         <material name="body" />
       </visual>
@@ -144,8 +139,7 @@
       <visual>
         <origin xyz="0 0 0"
-                rpy="${PI / 2.0} 0 0" />
+                rpy="0 0 0" />
         <geometry>
-          <cylinder length="0.025"
-                    radius="0.045" />
+          <mesh filename="package://kachaka_description/meshes/kachaka/left_tire.stl" scale="1.0 1.0 1.0"/>
         </geometry>
         <material name="tire" />

Commit message: fixed camera orientation in URDF

File: ros2/kachaka_description/urdf/_kachaka.urdf.xacro (robot description, xacro)
@@ -127,5 +127,5 @@
       <parent link="base_link" />
       <child link="camera_front_link" />
-      <origin rpy="-${PI / 2.0} 0 -${PI / 2.0}"
+      <origin rpy="0 0 0"
               xyz="${0.2196 - 0.01} 0 0.070" />
     </joint>
@@ -136,5 +136,5 @@
       <parent link="base_link" />
       <child link="camera_back_link" />
-      <origin rpy="-${PI / 2.0} 0 ${PI / 2.0}"
+      <origin rpy="0 0 ${PI}"
               xyz="${-0.150 + 0.01} 0 0.070" />
     </joint>
@@ -145,5 +145,5 @@
       <parent link="base_link" />
       <child link="tof_link" />
-      <origin rpy="-${PI / 4.0} 0 -${PI / 2.0}"
+      <origin rpy="0 -${PI / 4.0} 0"
               xyz="0.221 0.0 0.0418" />
     </joint>

Commit message: Fix mesh path

File: ros2/kachaka_description/urdf/_kachaka.urdf.xacro (robot description, xacro)
@@ -21,5 +21,5 @@
         <origin rpy="0 0 0" xyz="-0.150 -0.120 0.0"/>
         <geometry>
-          <mesh filename="package://kachaka_description/meshes/kachaka/body.stl"/>
+          <mesh filename="file://$(find kachaka_description)/meshes/kachaka/body.stl"/>
         </geometry>
         <material name="body" />
@@ -59,5 +59,5 @@
         <origin rpy="0 0 0" xyz="0 0 0"/>
         <geometry>
-          <mesh filename="package://kachaka_description/meshes/kachaka/right_tire.stl" scale="1.0 1.0 1.0"/>
+          <mesh filename="file://$(find kachaka_description)/meshes/kachaka/right_tire.stl" scale="1.0 1.0 1.0"/>
         </geometry>
         <material name="tire" />
@@ -99,5 +99,5 @@
                 rpy="0 0 0" />
         <geometry>
-          <mesh filename="package://kachaka_description/meshes/kachaka/left_tire.stl" scale="1.0 1.0 1.0"/>
+          <mesh filename="file://$(find kachaka_description)/meshes/kachaka/left_tire.stl" scale="1.0 1.0 1.0"/>
         </geometry>
         <material name="tire" />
@@ -173,5 +173,5 @@
       <visual>
         <geometry>
-          <mesh filename="package://kachaka_description/meshes/kachaka/solenoid.stl"
+          <mesh filename="file://$(find kachaka_description)/meshes/kachaka/solenoid.stl"
                 scale="1.0 1.0 1.0" />
         </geometry>
